File: Driver Motor PaP_V1.0/Driver Motor PaP_V1.0.kicad_pcb (KiCad board)
At the start: 2 copper layers, 27 parts, among them J1 Conn_01x02, J2 Conn_01x02, J3 Conn_01x02, J4 Conn_01x04, J5 Conn_01x01, J6 Conn_01x02, J7 Conn_01x02, U1 LM358, U2 LM358, U3 LM358

Commit message: PCB Driver Motor PaP
Parts:
- added C2: 100nF, Capacitor_SMD:C_0805_2012Metric_Pad1.15x1.40mm_HandSolder, F.Cu at (132.2, 89.2)
- added C3: 100nF, Capacitor_SMD:C_0805_2012Metric_Pad1.15x1.40mm_HandSolder, B.Cu at (154.2, 122.8)
- added C4: 100nF, Capacitor_SMD:C_0805_2012Metric_Pad1.15x1.40mm_HandSolder, F.Cu at (153.5, 117.8)
- added FID1: Fiducial, Fiducial:Fiducial_1mm_Mask2mm, F.Cu at (111.2, 122.8)
- C1: footprint Capacitor_THT:C_Radial_D6.3mm_H11.0mm_P2.50mm -> Capacitor_SMD:CP_Elec_6.3x5.4; moved to B.Cu
- D1: footprint LED_THT:LED_D3.0mm -> LED_SMD:LED_0805_2012Metric_Pad1.15x1.40mm_HandSolder
- H1, H2, H3, H4: footprint MountingHole:MountingHole_3mm_Pad -> MountingHole:MountingHole_3.2mm_M3
- J1, J2: footprint Connector_PinHeader_2.54mm:PinHeader_1x02_P2.54mm_Vertical -> TerminalBlock:TerminalBlock_bornier-2_P5.08mm
- J3: value Conn_01x02 -> Conn_01x03; footprint Connector_PinHeader_2.54mm:PinHeader_1x02_P2.54mm_Vertical -> Connector_Molex:Molex_KK-254_AE-6410-03A_1x03_P2.54mm_Vertical
- J4: value Conn_01x04 -> Conn_01x05; footprint Connector_PinHeader_2.54mm:PinHeader_1x04_P2.54mm_Vertical -> Connector_Molex:Molex_KK-254_AE-6410-05A_1x05_P2.54mm_Vertical
- R1: footprint Resistor_THT:R_Axial_DIN0207_L6.3mm_D2.5mm_P10.16mm_Horizontal -> Resistor_SMD:R_0805_2012Metric_Pad1.15x1.40mm_HandSolder
- U1, U2: footprint Package_DIP:DIP-8_W7.62mm -> Package_SO:SOIC-8_3.9x4.9mm_P1.27mm; moved to B.Cu
- U3: footprint Package_DIP:DIP-8_W7.62mm -> Package_SO:SOIC-8_3.9x4.9mm_P1.27mm
- moved J1 214.4 mm to (111.8, 105.0), turned to 270 degrees
- moved J7 208.2 mm to (131.7, 132.2), turned to 90 degrees
- moved J3 204.5 mm to (117.2, 90.0)
- moved H4 202.9 mm to (111.2, 131.2)
- moved JP7 198.8 mm to (121.0, 102.8), turned to 90 degrees
- moved J6 198.1 mm to (126.6, 132.2), turned to 270 degrees
- moved JP9 197.8 mm to (121.0, 117.0), turned to 90 degrees
- moved D1 195.8 mm to (113.0, 97.0), turned to 270 degrees
- moved JP8 194.6 mm to (121.0, 110.0), turned to 90 degrees
- moved JP2 181.1 mm to (154.5, 107.5), turned to 270 degrees
- moved C1 179.6 mm to (145.0, 122.8), turned to 180 degrees
- moved U1 177.8 mm to (132.0, 96.2), turned to 180 degrees
- moved JP1 176.4 mm to (154.5, 113.8), turned to 270 degrees
- moved A1 176.3 mm to (129.0, 115.8), turned to 90 degrees
- moved J2 175.5 mm to (143.2, 131.0)
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Connections:
- net /GNDMotor renamed GNDPWR
- net /VMotor renamed VPP
- U1 pad 5: Net-(J4-Pad2) -> Net-(J3-Pad2)
- U1 pad 6: Net-(JP5-Pad1) -> Net-(A1-Pad16)
- U1 pad 7: Net-(JP5-Pad1) -> Net-(A1-Pad16)
- U2 pad 5: Net-(J3-Pad2) -> Net-(J4-Pad2)
- U2 pad 6: Net-(A1-Pad16) -> Net-(JP5-Pad1)
- U2 pad 7: Net-(A1-Pad16) -> Net-(JP5-Pad1)
Routing:
- net GND: track 0.00 -> 78.0 mm, vias 0 -> 3
- net Net-(JP8-Pad1): track 0.00 -> 71.9 mm
- net Net-(JP5-Pad1): track 0.00 -> 69.0 mm
- net Net-(A1-Pad12): track 0.00 -> 61.8 mm
- net VCC: track 0.00 -> 36.2 mm, vias 0 -> 3
- net Net-(J4-Pad3): track 0.00 -> 35.6 mm
- net Net-(J3-Pad1): track 0.00 -> 35.4 mm
- net GNDPWR: track 0.00 -> 28.8 mm
- net Net-(A1-Pad15): track 0.00 -> 28.3 mm, vias 0 -> 1
- net Net-(A1-Pad11): track 0.00 -> 25.8 mm
- net Net-(J4-Pad2): track 0.00 -> 24.0 mm
- net Net-(A1-Pad10): track 0.00 -> 22.5 mm
- net Net-(J4-Pad1): track 0.00 -> 22.3 mm
- net Net-(J5-Pad1): track 0.00 -> 22.3 mm
- net Net-(A1-Pad4): track 0.00 -> 21.1 mm
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- added copper zone on 2-In1.Cu.GND, net GND
- added copper zone on B.Cu, net GND
- added copper zone on F.Cu, net GND
- added copper zone on 3-In2.Cu.VCC, net VCC
Other:
- board outline added: 60 x 50 mm
- copper layers 2 -> 4
- net class Default: clearance 0.2 -> 0.25; trace_width 0.25 -> 0.5; via_dia 0.8 -> 1.6; via_drill 0.4 -> 0.8
- rule trace_clearance: 0.2 -> 0.25
- board text added: "+"
- board text added: "."
- board text added: "1"
- board text added: "Autor: Mariano Campos"
- board text added: "CESE 8va Cohorte 2019"
- board text added: "Diseño Argentino"
- board text added: "Driver Motor PaP-V1.0"
- board text added: "M0"
- board text added: "M1"
- board text added: "M2"
- board text added: "Mínimos (10 Mils Mayer ) Grillas: 0,25 mm vías : 2mm ,agujeros 0,9 mm. Margen General: 0,25 mm Ancho de pista : 0,5 mm y 1,2 mm. Distancia a borde: 0,5 mm. Terminación HASL."
- board text added: "Pahse A"
- board text added: "Phase B"
- board text added: "Vcc"
- board text added: "Vmotor"
- board text added: "[ 2 ]"
- board text added: "[ 3 ]"
- board text added: "[ 4]"
- board text added: "[1 ]"
- board text added: "dir"
- board text added: "gnd"
- board text added: "stp"

Commit message: correcciones driver motor PaP v1.0
Other:
- board text added: "LED_PWR"
- board text added: "Mínimos (10 Mils Mayer ) Grillas: 0,25 mm. vías : 2mm ,agujeros 0,9 mm. Margen General: 0,25 mm. Ancho de pista : 0,5 mm y 1,2 mm. Distancia a borde: 0,5 mm. PCB espesor: 1,6mm. Terminación HASL."
- board text removed: "Mínimos (10 Mils Mayer ) Grillas: 0,25 mm vías : 2mm ,agujeros 0,9 mm. Margen General: 0,25 mm Ancho de pista : 0,5 mm y 1,2 mm. Distancia a borde: 0,5 mm. Terminación HASL."
